Commit message: fix navigation issue

File: omni_robot_description/robots/omni_robot_v2.urdf.xacro (robot description, xacro)
@@ -4,5 +4,5 @@
   <xacro:property name="M_PI" value="3.14159274" />
   <!-- xacro include file -->
-  <xacro:include filename="$(find omni_robot_description)/urdf/base/base_v1.urdf.xacro" />  <!--base-->
+  <xacro:include filename="$(find omni_robot_description)/urdf/base/base.urdf.xacro" />  <!--base-->
   <xacro:include filename="$(find omni_robot_description)/urdf/base_layer/base_layer.urdf.xacro" />  <!--base-->
   <xacro:include filename="$(find omni_robot_description)/urdf/camera/camera.urdf.xacro" />   <!--camera-->
@@ -15,8 +15,8 @@
   <!-- Base -->
   <link name="base_footprint" />
-  <!-- <xacro:base_v0 parent="base_footprint">
-    <origin xyz="0 0 0" rpy="0 0 0" />
-  </xacro:base_v0> -->
-  <xacro:base_v1 parent="base_footprint" xyz="0 0 0" rpy="0 0 ${-M_PI/2}" />
+  <xacro:base_v0 parent="base_footprint">
+    <origin xyz="0 0 0" rpy="0 0 ${-M_PI/2}" />
+  </xacro:base_v0>
+  <!-- <xacro:base_v1 parent="base_footprint" xyz="0 0 0" rpy="0 0 ${-M_PI/2}" /> -->
   <!-- Base Layer -->
   <!-- <xacro:base_layer prefix="first" parent="base_footprint" xyz="0 0 0.125" rpy="0 0 ${M_PI/2}" /> -->
@@ -24,5 +24,5 @@
   <!-- Wheel -->
   <!-- 1st wheel -->
-  <xacro:wheel_v0 prefix="first" parent="base_link_ext">
+  <xacro:wheel_v0 prefix="first" parent="base_link">
     <origin xyz="0 0.088 -0.01" rpy="0 0 3.141593" />
     <axis xyz="0 1 0" />
@@ -69,5 +69,5 @@
   </xacro:roller_v0>
   <!-- 2nd wheel -->
-  <xacro:wheel_v0 prefix="second" parent="base_link_ext">
+  <xacro:wheel_v0 prefix="second" parent="base_link">
     <origin xyz="-0.0762 -0.044 -0.01" rpy="0 0 5.235988" />
     <axis xyz="0 1 0" />
@@ -114,5 +114,5 @@
   </xacro:roller_v0>
   <!-- 3rd wheel -->
-  <xacro:wheel_v0 prefix="third" parent="base_link_ext">
+  <xacro:wheel_v0 prefix="third" parent="base_link">
     <origin xyz="0.0762 -0.044 -0.01" rpy="0 0 1.047197" />
     <axis xyz="0 1 0" />
@@ -167,5 +167,5 @@
   </xacro:camera_v0>
   <!-- camera bracket-->
-  <xacro:camera_bracket_v0 prefix="main" parent="base_link_ext">
+  <xacro:camera_bracket_v0 prefix="main" parent="base_link">
     <origin xyz="0 0 0.039" rpy="0 0 1.570796" />
     <axis xyz="0 0 1" />
@@ -183,4 +183,6 @@
     </plugin>
   </gazebo>
+  <!-- Base -->
+  <xacro:base_gazebo_v0 />
   <!-- Wheel -->
   <xacro:wheel_gazebo_v0 prefix="first" />
